Commit message: .dae file directory changed

File: p3dx_description/urdf/sensors/asus_camera.urdf.xacro (robot description, xacro)
@@ -24,5 +24,5 @@
         <geometry>
           <!--box size="0.035 0.185 0.025"/-->
-          <mesh filename="package://mbot_description/meshes/sensors/asus_camera_simple.dae"/>
+          <mesh filename="package://p3dx_description/meshes/sensors/asus_camera_simple.dae"/>
         </geometry>
       </visual>
