Commit message: put arucos at the same height than robot

File: p3dx_description/urdf/pioneer3dx_with_asus_camera.xacro (robot description, xacro)
@@ -10,6 +10,6 @@
 		<parent link="top_plate" />
 		<child link="camera_model_link" />
-		<!--<origin xyz="0.12 0 0.05" rpy="0 0.8 0" /> -->
-		<origin xyz="0.12 0 0.02" rpy="0 -0.2 0" />
+		<!--<origin xyz="0.12 0 0.05" rpy="0 0.275 0" /> -->
+		<origin xyz="0.12 0 0.02" rpy="0 0 0" />
 	</joint>
 </robot>
