Commit message: new launch to launch gazebo and rviz in once

File: p3dx_description/urdf/materials.xacro (robot description, xacro)
@@ -18,5 +18,5 @@
  -->
 <!-- NOTE: this materials are for rviz visualization, for gazebo visualization check: pioneer3dx.gazebo -->
-<robot name="pioneer3dx" xmlns:xacro="http://www.ros.org/xacro">
+<robot name="pioneer3dx" xmlns:xacro="http://wiki.ros.org/xacro">
     <material name="ChassisRed">
         <color rgba="0.8 0.0 0.0 1.0"/>

File: p3dx_description/urdf/pioneer3dx.xacro (robot description, xacro)
@@ -17,5 +17,5 @@
 NOTE: Migration to ROS kinetic and gazebo 7 performed by Oscar Lima olima@isr.tecnico.ulisboa.pt
  -->
-<robot name="pioneer3dx" xmlns:xacro="http://www.ros.org/xacro">
+<robot name="pioneer3dx" xmlns:xacro="http://wiki.ros.org/xacro">
 <!-- import the pioneer 3dx's wheels -->
 <xacro:include filename="$(find p3dx_description)/urdf/pioneer3dx_wheel.xacro" />
@@ -39,10 +39,22 @@
         </geometry>
     </collision>
-    <inertial>
+    <!--inertial>
         <mass value="3.5" />
         <origin xyz="-0.05 0 0" />
         <inertia ixx="1" ixy="0" ixz="0" iyy="1" iyz="0" izz="1" />
-    </inertial>
-</link>
+    </inertial-->
+</link>
+<link name="base_link_dummy">
+    <inertial>
+        <mass value="3.5" />
+        <origin xyz="-0.05 0 0" />
+        <inertia ixx="1" ixy="0" ixz="0" iyy="1" iyz="0" izz="1" />
+    </inertial>
+</link>
+<joint name="base_link_inertial_joint" type="fixed">
+    <origin xyz="0 0 0" rpy="0 0 0" />
+    <parent link="base_link" />
+    <child link="base_link_dummy" />
+</joint>
 <!-- top_plate -->
 <link name="top_plate">

File: p3dx_description/urdf/pioneer3dx_wheel.xacro (robot description, xacro)
@@ -17,5 +17,5 @@
 NOTE: Migration to ROS kinetic and gazebo 7 performed by Oscar Lima olima@isr.tecnico.ulisboa.pt
  -->
-<robot xmlns:xacro="http://www.ros.org/xacro">
+<robot xmlns:xacro="http://wiki.ros.org/xacro">
 <!-- macro to generate pioneer wheels (right/left hubcap + wheel) -->
 <xacro:macro name="p3dx_wheel" params="suffix parent reflect">
