Commit message: changing <box size='0 0 0' by<box size='0.0001 0.0001 0.0001' />

File: p3dx_description/urdf/pioneer3dx.xacro (robot description, xacro)
@@ -83,5 +83,5 @@
         <origin xyz="0 0 0" rpy="0 0 0" />
         <geometry>
-            <box size="0 0 0" />
+            <box size="0.0001 0.0001 0.0001" />
         </geometry>
     </collision>
@@ -113,5 +113,5 @@
         <origin xyz="0 0 0" rpy="0 0 0" />
         <geometry>
-            <box size="0 0 0" />
+            <box size="0.0001 0.0001 0.0001" />
         </geometry>
     </collision>
@@ -173,5 +173,5 @@
         <origin rpy="0 0 0" xyz="0 0 0" />
         <geometry>
-            <box size="0 0 0" />
+            <box size="0.0001 0.0001 0.0001" />
         </geometry>
     </collision>

File: p3dx_description/urdf/pioneer3dx_wheel.xacro (robot description, xacro)
@@ -65,5 +65,5 @@
             <origin xyz="0 0 0" rpy="0 0 0" />
             <geometry>
-                <box size="0 0 0" />
+                <box size="0.0001 0.0001 0.0001" />
             </geometry>
         </collision>

Commit message: last commit well done

File: p3dx_description/urdf/pioneer3dx.xacro (robot description, xacro)
@@ -167,5 +167,5 @@
 </link>
 <joint name="center_wheel_joint" type="fixed">
-    <origin xyz="-0.0035 0 -0.001" rpy="0 0 0"/>
+    <origin xyz="0 0 0" rpy="0 0 0"/>
     <parent link="center_wheel"/>
     <child link="center_hubcap"/>
